Commit message: rotated camera 180 degrees

File: urdf/panda_with_rs.urdf (robot description, URDF)
Before this commit: robot panda, 18 links, 17 joints
Joints:
- joint realsense_joint: origin xyz=0.03 -0.03 0.05 rpy=0 -1.57079632679 -0.785398163397 -> xyz=0.03 -0.03 0.05 rpy=0 -1.57079632679 2.3561944901

File: urdf/panda_with_rs.xacro (robot description, xacro)
@@ -7,5 +7,5 @@
   <!-- Here we include the end-effector by setting the parameters -->
   <xacro:realsense-rs200 prefix="" parent="panda_link8">
-    <origin xyz="0.03 -0.03 0.05" rpy="0 ${-pi/2} ${-pi/4}" />
+    <origin xyz="0.03 -0.03 0.05" rpy="0 ${-pi/2} ${3*pi/4}" />
   </xacro:realsense-rs200>
 </robot>

File: urdf/panda_with_rs_PYBULLET.urdf (robot description, URDF)
Before this commit: robot panda, 18 links, 17 joints
Joints:
- joint realsense_joint: origin xyz=0.03 -0.03 0.05 rpy=0 -1.57079632679 -0.785398163397 -> xyz=0.03 -0.03 0.05 rpy=0 -1.57079632679 2.3561944901
